File: 2DMega/2DMega.sch (KiCad schematic (older format))
At the start: 51 parts, among them J1 Conn_01x06_Male, J2 Conn_01x06_Female, J3 Conn_02x03_Odd_Even, J4 Conn_01x06_Male, J5 Conn_01x06_Female, P1 Power, P10 CONN_01X01, P11 CONN_01X01, P12 CONN_01X01, P13 CONN_01X01, P2 Analog, P3 Analog, P4 Digital, P5 PWM, P6 PWM, P7 Communication, P8 CONN_01X01, P9 CONN_01X01, SW1 SW_SPST, U1 HDSP-A153

Commit message: As built
Parts:
- R1, R10, R11, R3, R5, R6, R7, R8: value 200 -> 300
Other:
- note added: "EAST"
- note added: "NORTH"
- note added: "SOUTH"
- note added: "WEST"
Changed lines of the file:
@@
 P 2850 5450
 F 0 "R10" H 2920 5496 50  0000 L CNN
-F 1 "200" H 2920 5405 50  0000 L CNN
+F 1 "300" H 2920 5405 50  0000 L CNN
 F 2 "Resistor_SMD:R_0805_2012Metric_Pad1.20x1.40mm_HandSolder" V 2780 5450 50  0001 C CNN
 F 3 "~" H 2850 5450 50  0001 C CNN
@@
 P 2250 5650
 F 0 "R5" H 2320 5696 50  0000 L CNN
-F 1 "200" H 2320 5605 50  0000 L CNN
+F 1 "300" H 2320 5605 50  0000 L CNN
 F 2 "Resistor_SMD:R_0805_2012Metric_Pad1.20x1.40mm_HandSolder" V 2180 5650 50  0001 C CNN
 F 3 "~" H 2250 5650 50  0001 C CNN
@@
 P 2550 5550
 F 0 "R7" H 2620 5596 50  0000 L CNN
-F 1 "200" H 2620 5505 50  0000 L CNN
+F 1 "300" H 2620 5505 50  0000 L CNN
 F 2 "Resistor_SMD:R_0805_2012Metric_Pad1.20x1.40mm_HandSolder" V 2480 5550 50  0001 C CNN
 F 3 "~" H 2550 5550 50  0001 C CNN
@@
 P 1950 5750
 F 0 "R3" H 2020 5796 50  0000 L CNN
-F 1 "200" H 2020 5705 50  0000 L CNN
+F 1 "300" H 2020 5705 50  0000 L CNN
 F 2 "Resistor_SMD:R_0805_2012Metric_Pad1.20x1.40mm_HandSolder" V 1880 5750 50  0001 C CNN
 F 3 "~" H 1950 5750 50  0001 C CNN
@@
 P 1650 5850
 F 0 "R1" H 1720 5896 50  0000 L CNN
-F 1 "200" H 1720 5805 50  0000 L CNN
+F 1 "300" H 1720 5805 50  0000 L CNN
 F 2 "Resistor_SMD:R_0805_2012Metric_Pad1.20x1.40mm_HandSolder" V 1580 5850 50  0001 C CNN
 F 3 "~" H 1650 5850 50  0001 C CNN
@@
 P 2850 5950
 F 0 "R11" H 2920 5996 50  0000 L CNN
-F 1 "200" H 2920 5905 50  0000 L CNN
+F 1 "300" H 2920 5905 50  0000 L CNN
 F 2 "Resistor_SMD:R_0805_2012Metric_Pad1.20x1.40mm_HandSolder" V 2780 5950 50  0001 C CNN
 F 3 "~" H 2850 5950 50  0001 C CNN
@@
 P 2550 6050
 F 0 "R8" H 2620 6096 50  0000 L CNN
-F 1 "200" H 2620 6005 50  0000 L CNN
+F 1 "300" H 2620 6005 50  0000 L CNN
 F 2 "Resistor_SMD:R_0805_2012Metric_Pad1.20x1.40mm_HandSolder" V 2480 6050 50  0001 C CNN
 F 3 "~" H 2550 6050 50  0001 C CNN
@@
 P 2250 6150
 F 0 "R6" H 2320 6196 50  0000 L CNN
-F 1 "200" H 2320 6105 50  0000 L CNN
+F 1 "300" H 2320 6105 50  0000 L CNN
 F 2 "Resistor_SMD:R_0805_2012Metric_Pad1.20x1.40mm_HandSolder" V 2180 6150 50  0001 C CNN
 F 3 "~" H 2250 6150 50  0001 C CNN
@@
 Wire Wire Line
 	6250 2950 6250 2850
+Text Notes 5150 1250 0    50   ~ 0
+NORTH
+Text Notes 5150 2800 0    50   ~ 0
+SOUTH
+Text Notes 6800 2800 0    50   ~ 0
+WEST
+Text Notes 6850 1250 0    50   ~ 0
+EAST
 $EndSCHEMATC
