File: 3DESPWrover/3DESPWrover.kicad_pcb (KiCad board)
At the start: 2 copper layers, 40 x 40 mm, 23 parts, among them J1 Conn_01x05_Male, J2 Conn_01x03_Female, J3 Conn_02x03_Odd_Even, J4 Conn_02x07_Odd_Even, SW1 SW_Push, SW2 SW_Push, U1 ESP32-S2-WROVER

Commit message: Correction to 3.3v regulator connection
Parts:
- moved NT1 0.44 mm to (230.9, 85.8)
- moved L1 0.36 mm to (230.9, 85.8)
Connections:
- J2 pad 2: /Vout -> GND
- J2 pad 3: GND -> /Vout
Routing:
- net GND: track 7.56 -> 9.39 mm
- net /Vout: track 9.42 -> 10.3 mm
Other:
- board text added: "3.3V"
- board text added: "D+"
- board text added: "D-"
- board text added: "D10"
- board text added: "D11"
- board text added: "D12"
- board text added: "D13"
- board text added: "D14"
- board text added: "D15"
- board text added: "D16"
- board text added: "D5"
- board text added: "D6"
- board text added: "D7"
- board text added: "D8"
- board text added: "D9"
- board text added: "G"
- board text added: "GND"
- board text added: "VCC"
