File: 3DESPWrover/3DESPWrover.kicad_sch (KiCad schematic)
At the start: 30 parts, among them J1 Conn_01x04_Male, J3 Conn_02x03_Odd_Even, J4 Conn_02x07_Odd_Even, SW1 SW_Push, SW2 SW_Push, U1 ESP32-S2-WROVER, U2 K78xxJT-500R3

Commit message: Sent cube to assembly manufacture, soldered PressureSensors, created test sketch for pressure sensors for arduino uno
Parts:
- D2: MPN (none) -> SS13
- J1: MPN (none) -> 0022052041
- J3: MPN (none) -> SSW-103-01-F-D
- R1, R10, R11, R12, R2, R5, R6, R7, R8, R9: MPN (none) -> Resistor, 510.0Ω, 0603 SMD
- R3, R4: MPN Resistor, 10.0kΩ, 0805 SMD -> Resistor, 10.0kΩ, 0805 SMD
- U1: MPN (none) -> DFR0743-WROVER
- U2: MPN (none) -> K7803JT-500R3
Changed lines of the file:
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@@
+      (effects (font (size 1.27 1.27)) hide)
+    )
+    (property "MPN" "SSW-103-01-F-D" (id 4) (at 153.67 90.17 0)
       (effects (font (size 1.27 1.27)) hide)
     )
@@
       (effects (font (size 1.27 1.27)) hide)
     )
-    (property "MPN" "Resistor, 10.0kΩ, 0805 SMD " (id 4) (at 224.79 17.78 0))
+    (property "MPN" "Resistor, 10.0kΩ, 0805 SMD" (id 4) (at 224.79 17.78 0))
     (pin "1")
     (pin "2")
@@
       (effects (font (size 1.27 1.27)) hide)
     )
-    (property "MPN" " Resistor, 10.0kΩ, 0805 SMD " (id 4) (at 26.67 102.87 0))
+    (property "MPN" "Resistor, 10.0kΩ, 0805 SMD" (id 4) (at 26.67 102.87 0))
     (pin "1")
     (pin "2")
@@
       (effects (font (size 1.27 1.27)) hide)
     )
+    (property "MPN" "Resistor, 510.0Ω, 0603 SMD" (id 4) (at 211.455 85.09 0)
+      (effects (font (size 1.27 1.27)) hide)
+    )
     (pin "1")
     (pin "2")
@@
       (effects (font (size 1.27 1.27)) hide)
     )
+    (property "MPN" "K7803JT-500R3" (id 4) (at 261.62 23.495 0)
+      (effects (font (size 1.27 1.27)) hide)
+    )
     (pin "1")
     (pin "2")
@@
     )
     (property "Datasheet" "https://www.espressif.com/sites/default/files/documentation/esp32-s2-wroom_esp32-s2-wroom-i_datasheet_en.pdf" (id 3) (at 35.56 77.47 0)
+      (effects (font (size 1.27 1.27)) hide)
+    )
+    (property "MPN" "DFR0743-WROVER" (id 4) (at 43.18 57.15 0)
       (effects (font (size 1.27 1.27)) hide)
     )
@@
       (effects (font (size 1.27 1.27)) hide)
     )
+    (property "MPN" "Resistor, 510.0Ω, 0603 SMD" (id 4) (at 187.325 90.17 0)
+      (effects (font (size 1.27 1.27)) hide)
+    )
     (pin "1")
     (pin "2")
@@
       (effects (font (size 1.27 1.27)) hide)
     )
+    (property "MPN" "Resistor, 510.0Ω, 0603 SMD" (id 4) (at 211.455 90.17 0)
+      (effects (font (size 1.27 1.27)) hide)
+    )
     (pin "1")
     (pin "2")
@@
       (effects (font (size 1.27 1.27)) hide)
     )
+    (property "MPN" "Resistor, 510.0Ω, 0603 SMD" (id 4) (at 211.455 87.63 0)
+      (effects (font (size 1.27 1.27)) hide)
+    )
     (pin "1")
     (pin "2")
@@
     )
     (property "Datasheet" "~" (id 3) (at 211.455 92.71 0)
+      (effects (font (size 1.27 1.27)) hide)
+    )
+    (property "MPN" "Resistor, 510.0Ω, 0603 SMD" (id 4) (at 211.455 92.71 0)
       (effects (font (size 1.27 1.27)) hide)
     )
@@
       (effects (font (size 1.27 1.27)) hide)
     )
+    (property "MPN" "0022052041" (id 4) (at 133.35 35.56 0)
+      (effects (font (size 1.27 1.27)) hide)
+    )
     (pin "1")
     (pin "2")
@@
       (effects (font (size 1.27 1.27)) hide)
     )
+    (property "MPN" "Resistor, 510.0Ω, 0603 SMD" (id 4) (at 187.325 87.63 0)
+      (effects (font (size 1.27 1.27)) hide)
+    )
     (pin "1")
     (pin "2")
@@
       (effects (font (size 1.27 1.27)) hide)
     )
+    (property "MPN" "Resistor, 510.0Ω, 0603 SMD" (id 4) (at 211.455 95.25 0)
+      (effects (font (size 1.27 1.27)) hide)
+    )
     (pin "1")
     (pin "2")
@@
       (effects (font (size 1.27 1.27)) hide)
     )
+    (property "MPN" "Resistor, 510.0Ω, 0603 SMD" (id 4) (at 187.325 95.25 0)
+      (effects (font (size 1.27 1.27)) hide)
+    )
     (pin "1")
     (pin "2")
@@
       (effects (font (size 1.27 1.27)) hide)
     )
+    (property "MPN" "Resistor, 510.0Ω, 0603 SMD" (id 4) (at 187.325 85.09 0)
+      (effects (font (size 1.27 1.27)) hide)
+    )
     (pin "1")
     (pin "2")
@@
       (effects (font (size 1.27 1.27)) hide)
     )
+    (property "MPN" "Resistor, 510.0Ω, 0603 SMD" (id 4) (at 187.325 92.71 0)
+      (effects (font (size 1.27 1.27)) hide)
+    )
     (pin "1")
     (pin "2")
@@
       (effects (font (size 1.27 1.27)) hide)
     )
+    (property "MPN" "SS13" (id 4) (at 246.38 20.955 0)
+      (effects (font (size 1.27 1.27)) hide)
+    )
