File: 3DESPWroverB/3DESPWroverB.sch (KiCad schematic (older format))
At the start: 18 parts, among them J1 Conn_02x07_Odd_Even, J10 Conn_02x03_Odd_Even, J11 Conn_01x01, J12 Conn_01x01, J13 Conn_01x01, J14 Conn_01x01, J15 Conn_01x01, J16 Conn_01x01, J17 Conn_01x01, J18 Conn_01x01, J2 Conn_01x01, J3 Conn_01x01, J4 Conn_01x01, J5 Conn_01x01, J6 Conn_01x01, J7 Conn_01x01, J8 Conn_01x01, J9 Conn_01x01

Commit message: Some components replaced by SMD versions
Parts:
- J1: footprint Custom:TE_Micromatch_2,54_14 -> Custom:TE_Micromatch_2,54_14_SMD
Changed lines of the file:
@@
 F 0 "J1" H 1850 2017 50  0000 C CNN
 F 1 "Conn_02x07_Odd_Even" H 1850 1926 50  0000 C CNN
-F 2 "Custom:TE_Micromatch_2,54_14" H 1800 1500 50  0001 C CNN
+F 2 "Custom:TE_Micromatch_2,54_14_SMD" H 1800 1500 50  0001 C CNN
 F 3 "~" H 1800 1500 50  0001 C CNN
 	1    1800 1500
