File: PressureSensors/PressureSensors.kicad_pcb (KiCad board)
At the start: 2 copper layers, 40 x 40 mm, 27 parts, among them IC1 BD733L2FP3-CE2, J1 Conn_02x03_Odd_Even, U1 LPS22HB, U2 LPS22HB, U3 LPS22HB, U4 LPS22HB, U5 PCA9543AD

Commit message: Before PC swap
Parts:
- U1, U2, U3, U4: value LPS22HB -> LPS33HW; footprint Custom:LPS22HBTR -> Custom:LPS33HW
Routing:
- net +3V3: track 81.7 -> 97.7 mm
- net GND: track 51.8 -> 42.2 mm
- net /SCL0: track 70.8 -> 68.2 mm
- net /SDA0: track 49.0 -> 46.5 mm
- net /SDA1: track 64.1 -> 61.6 mm
- net unconnected-(U4-Pad7): track 2.24 -> 0.00 mm
- net unconnected-(U1-Pad7): track 2.22 -> 0.00 mm
- net unconnected-(U3-Pad7): track 2.20 -> 0.00 mm
- net unconnected-(U2-Pad7): track 2.19 -> 0.00 mm
- net /SCL1: track 71.1 -> 69.2 mm
Other:
- board text added: "MOZART V1.5 REAL ITU"
- board text removed: "MOZART V1.1 REAL ITU"
